File: PLC.kicad_sch (KiCad schematic)
At the start: 118 parts, among them J1 TB_1X2, J10 TB_1X2, J2 TB_1X3, J3 TB_1X2, J4 TB_1X2, J5 TB_1X2, J6 TB_1X2, J7 TB_1X2, J8 TB_1X2, J9 TB_1X2, K1 RELAY_C, K2 RELAY_C, K3 RELAY_C, K4 RELAY_C, K5 RELAY_C, K6 RELAY_C, Q1 MMBT3904, Q2 MMBT3904, Q3 MMBT3904, Q4 MMBT3904, Q5 MMBT3904, Q6 MMBT3904, Q7 AO3401A, Q8 AO3401A, Q9 AO3401A, U1 LM2594M-5.0, U2 LM2594M-3.3, U3 LM321MF_NOPB, U5 LM321MF_NOPB

Commit message: new
Parts:
- removed D1, D2, D7: SS210, SS210:DIOM4336X265N, symbol SS210:SS210
- removed D10, D11, D12, D13, D14, D15: 1N4148, Diode_THT:D_DO-35_SOD27_P7.62mm_Horizontal, symbol Diode:1N4148
- removed D8, D9: BZT52C3V3-7-F, BZT52C3V3-7-F:SOD3715X135N, symbol BZT52C3V3-7-F:BZT52C3V3-7-F
- removed J2: TB_1X3, EESTN5:BORNERA3_AZUL, symbol EESTN5:TB_1X3
- removed J3, J4, J5, J6, J7, J8: TB_1X2, EESTN5:BORNERA2, symbol EESTN5:TB_1X2
- removed OK1, OK2, OK3, OK4, OK5, OK6: PC817, PC817X2NIP0F:SOP254P975X460-4N, symbol PC817:PC817
- removed Q1, Q2, Q3, Q4, Q5, Q6: MMBT3904, Package_TO_SOT_SMD:SOT-23, symbol Transistor_BJT:MMBT3904
- removed R30, R31: R, EESTN5:R_0805, symbol Device:R
- removed U3, U5: LM321MF_NOPB, LM321MF_NOPB:SOT95P280X145-5N, symbol LM321MF_NOPB:LM321MF_NOPB
- added C10, C11, C12: C, Capacitor_SMD:C_0805_2012Metric_Pad1.18x1.45mm_HandSolder, symbol Device:C
- added D1, D2: 1N5822, Diode_THT:D_DO-201AD_P15.24mm_Horizontal, symbol Diode:1N5822
- added D10, D11, D12, D13, D14, D19: 1N4007, Diode_THT:D_DO-41_SOD81_P10.16mm_Horizontal, symbol Diode:1N4007
- added J11, J3, J4, J5, J6, J7: Salida, EESTN5:BORNERA3_AZUL, symbol Connector:Screw_Terminal_01x03
- added J12, J13, J2: TB_1X2, EESTN5:BORNERA2, symbol EESTN5:TB_1X2
- added J8: Screw_Terminal_01x04, Library:Bornera_4, symbol EESTN5:Screw_Terminal_01x04
- added JP1: Jumper, EESTN5:Jumper_Alto, symbol EESTN5:Jumper
- added Q1, Q10, Q2, Q3, Q4, Q5: 2N3904, Package_TO_SOT_SMD:SOT-23_Handsoldering, symbol Transistor_BJT:2N3904
- added R44: 220, EESTN5:RES0.3, symbol Device:R
- added R45: 1k, Resistor_SMD:R_1210_3225Metric_Pad1.30x2.65mm_HandSolder, symbol Device:R
- added U10, U13, U14, U15, U16, U17, U3, U4, U6, U7, U8, U9: PC817, Package_DIP:DIP-4_W7.62mm, symbol EESTN5:PC817
- added U11: BluePill, EESTN5:BluePill, symbol EESTN5:BluePill
- added U12: SN74HC541PWR, SN74HC541N:DIP254P762X508-20, symbol SN74HC14PWR:SN74HC14PWR
- added U5: SN74HC14PWR, SN74HC14N:DIP794W45P254L1969H508Q14, symbol SN74HC14PWR:SN74HC14PWR
- C1, C4: value CP -> 470uF
- C2, C5: value C -> 1uF; footprint (none) -> Capacitor_SMD:C_0805_2012Metric_Pad1.18x1.45mm_HandSolder
- C3, C6: value CP -> 220uF
- C7, C8, C9: footprint (none) -> Capacitor_SMD:C_0805_2012Metric_Pad1.18x1.45mm_HandSolder
- J1: value TB_1X2 -> 24V
- K1, K2, K3, K4, K5, K6: footprint SRD-24VDC-SL-C:RELAY_SRD-24VDC-SL-C -> EESTN5:Relay_C
- L1, L2: value L -> 68uH; footprint (none) -> Inductor_SMD:L_Bourns_SRR1260
- LED1: footprint (none) -> LED_SMD:LED_0805_2012Metric
- LED2, LED3, LED4, LED5, LED6, LED7: footprint (none) -> EESTN5:led_5mm_green
- R1: value R -> 1K
- R10, R2, R4, R6, R8: value R -> 220; footprint EESTN5:R_0805 -> EESTN5:RES0.3
- R11, R3, R5, R7, R9: value R -> 1k; footprint EESTN5:R_0805 -> Resistor_SMD:R_1210_3225Metric_Pad1.30x2.65mm_HandSolder
- R12, R15, R17, R19, R21, R23: footprint EESTN5:R_0805 -> EESTN5:RES0.3
- R32, R33, R34, R35, R38, R39: footprint Resistor_THT:R_Axial_DIN0309_L9.0mm_D3.2mm_P20.32mm_Horizontal -> EESTN5:R_0805
Connections:
- net 5v1 is gone; now on an unnamed net: D6.C
- net Earth: now also D3.A, D6.A, LED2.2 (K), LED3.2 (K), LED4.2 (K), LED5.2 (K), LED6.2 (K), LED7.2 (K), D1.1 (K), D1.2 (A), Q1.1 (E), Q10.1 (E), Q2.1 (E), Q3.1 (E), Q4.1 (E), Q5.1 (E), U12.7 (GND), U13.2, U13.3, U14.2, U14.3, U15.2, U15.3, U16.2, U16.3, U17.2, U17.3, U3.2, U3.3, U5.7 (GND); no longer C1.1, C2.1, D4.A, R12.1, R14.2, R17.1, R19.2, R2.1, R22.1, R24.2, R27.1, R29.2, R5.2, R7.1, R9.2, U1.7 (VIN)
- net VCC: now also C7.2, C8.2, C9.2, R13.2, R16.2, R18.2, R20.2, R22.2, R24.2, C10.2, C11.2, C12.2, U12.14 (VCC), U5.14 (VCC)
- net at F1.2: now also D2.2 (A); no longer D3.A
- net at L1.1, U1.8 (OUT): now also D3.C; no longer D4.C
- net at K6.2: now also D19.1 (K), Q10.3 (C); no longer LED7.2 (K)
- net at K1.1: now also J3.3 (Pin_3)
- net at K1.2: now also D10.1 (K), Q1.3 (C); no longer LED2.2 (K)
- net at K1.3: now also J3.2 (Pin_2)
- net at K1.4: now also J3.1 (Pin_1)
- net at R9.1: now also Q4.2 (B); no longer R10.1
- net at R12.2: now also U3.1; no longer R13.1
- net at K4.2: now also D13.1 (K), Q4.3 (C); no longer LED5.2 (K)
- net at R10.2: now also U10.1
- net 6Y hc14: now reaches R29.1
- net 6Y hc14: now also U12.13 (6A), U5.12 (6Y)
- net at R27.2: now also LED5.1 (A); no longer R28.1
- net at R5.1: now also Q2.2 (B); no longer R4.1
- net at R4.2: now also U7.1
- net at R17.2: now also U14.1; no longer R18.1
- net at R21.2: now also U16.1; no longer LED5.1 (A)
- net at K4.1: now also J6.3 (Pin_3)
- net at K4.3: now also J6.2 (Pin_2)
- net at LED3.1 (A): now also R25.2; no longer R11.2
- net at K2.2: now also D11.1 (K), Q2.3 (C); no longer LED3.2 (K)
- net at LED4.1 (A): now also R26.2; no longer R16.2
- net at K3.2: now also D12.1 (K), Q3.3 (C); no longer LED4.2 (K)
- net at R3.1: now also Q1.2 (B); no longer R2.2
- net IN6: now reaches R23.1
- net IN6: now also J2.2; no longer R22.2
- net at R23.2: now also U17.1
- net at K3.1: now also J5.3 (Pin_3)
- net at K3.3: now also J5.2 (Pin_2)
- net at K6.1: now also J11.3 (Pin_3)
- net at K6.3: now also J11.2 (Pin_2)
- net 1A hc14: now reaches C7.1
- net 1A hc14: now also R13.1, U3.4, U5.1 (1A)
- net at K5.1: now also J7.3 (Pin_3)
- net at K5.2: now also D14.1 (K), Q5.3 (C); no longer LED6.2 (K)
- net at K5.3: now also J7.2 (Pin_2)
- net at K5.4: now also J7.1 (Pin_1)
- net 1Y hc14: now reaches R14.1
- net 1Y hc14: now also U12.1 (1A), U5.2 (1Y); no longer R15.1
- net at C4.1, C5.1, U2.7 (VIN): now also D4.C; no longer D5.C
- net at R3.2: now also U6.3
- net 4A hc14: now reaches R20.1
- net 4A hc14: now also C10.1, U15.4, U5.9 (4A); no longer R19.1
- net at R28.2: now also LED6.1 (A)
- net 2Y hc14: now reaches R25.1
- net 2Y hc14: now also U12.3 (2A), U5.4 (2Y); no longer R24.1
- net at LED7.1 (A): now also R29.2
- net at R6.2: now also U8.1; no longer LED2.1 (A)
- net at R15.2: now also U13.1
- net at K3.4: now also J5.1 (Pin_1)
- net at K2.1: now also J4.3 (Pin_3)
- net at K2.3: now also J4.2 (Pin_2)
- net at R7.2: now also U8.3; no longer R8.1
- net 3A hc14: now reaches C9.1
- net 3A hc14: now also R18.1, U14.4, U5.5 (3A)
- net at K2.4: now also J4.1 (Pin_1)
- net 2A hc14: now reaches C8.1
- net 2A hc14: now also R16.1, U13.4, U5.3 (2A)
- net at R8.2: now also U9.1
- net at K6.4: now also J11.1 (Pin_1)
- net at K4.4: now also J6.1 (Pin_1)
- net +5V: no longer names the net of C3.1, D5.A, L1.2, U1.4 (FB)
- net +5V: now also D4.A; no longer D6.A
- net 24V renamed 5V
- net 5V: now also D5.C, D10.2 (A), D11.2 (A), D12.2 (A), D13.2 (A), D14.2 (A), D19.2 (A), U10.4, U11.18 (5V), U4.4, U6.4, U7.4, U8.4, U9.4; no longer D3.C, R11.1, R16.1, R21.1, R26.1, R6.1
- new net: R44.2, U4.1
- new net: R45.2, U4.3
- new net: Q10.2 (B), R45.1
- new net: R19.2, U15.1
- new net: R5.2, U7.3
- new net: R2.2, U6.1
- new net: LED2.1 (A), R14.2
- new net: J8.1 (Pin_1), JP1.1 (A)
- new net: J8.2 (Pin_2), JP1.2 (B)
- new net: J8.3 (Pin_3), U11.7 (PA10)
- new net: J8.4 (Pin_4), U11.6 (PA9)
- new net: Q3.2 (B), R7.1
- new net: C1.1, C2.1, D2.1 (K), U1.7 (VIN)
- new net: R11.2, U10.3
- new net: Q5.2 (B), R11.1
- new net: R9.2, U9.3
- new net 3Y hc14: R26.1, U12.5 (3A), U5.6 (3Y)
- new net 4Y hc14: R27.1, U12.9 (4A), U5.8 (4Y)
- new net 5A hc14: C11.1, R22.1, U16.4, U5.11 (5A)
- new net 5Y hc14: R28.1, U12.11 (5A), U5.10 (5Y)
- new net 6A hc14: C12.1, R24.1, U17.4, U5.13 (6A)
- new net GND: U10.2, U11.19 (GND), U11.39 (GND), U11.40 (GND), U4.2, U6.2, U7.2, U8.2, U9.2
- new net IN1: J13.1, R12.1
- new net IN2: J13.2, R15.1
- new net IN3: J12.1, R17.1
- new net IN4: J12.2, R19.1
- new net IN5: J2.1, R21.1
- new net PA0: R8.1, U11.25 (PA0)
- new net PA01: R10.1, U11.26 (PA1)
- new net PA02: R44.1, U11.27 (PA2)
- new net PB07: R2.1, U11.15 (PB7)
- new net PB08: R4.1, U11.16 (PB8)
- new net PB09: R6.1, U11.17 (PB9)
- no-connect marks 6 -> 0
Other:
- note added: "04/10/2025 (MM/DD/YYYY)"
- note added: "04/18/2025 (MM/DD/YYYY)"
- note added: "COM"
- note added: "DE"
- note added: "Digital inputs"
- note added: "NA"
- note added: "NC"
- note added: "RE"
- note added: "RX"
- note added: "Rele"
- note added: "STM32"
- note added: "TX"
- note removed: "4/10/2025 (MM/DD/YYYY)"
- moved on the sheet: C1, C2, C3, C4, C5, C6, D16, D17, D18, F1, J1, J10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
